Commit message: Lasers do LIDAR saindo do centro do LIDAR

File: src/roomba_bot/description/lidar.xacro (robot description, xacro)
@@ -5,10 +5,9 @@
         <parent link="chassis_link"/>
         <child link="laser_frame"/>
-        <origin xyz="0.17425 0.0 0.03347" rpy="0.0 0.0 0.0"/>
+        <origin xyz="0.17425 0.0 0.09634" rpy="0.0 0.0 0.0"/>
     </joint>
     <!-- Adding LIDAR properties -->
     <link name="laser_frame">
         <visual>
-            <origin xyz="0.0 0.0 0.0588"/>
             <geometry>
                 <cylinder radius="0.0343" length="0.0588" />
@@ -22,5 +21,5 @@
         </collision>
         <xacro:inertial_cylinder mass="0.5" length="0.0588" radius="0.0343">
-            <origin xyz="0 0 0" rpy="0.0 0.0 0.0" />
+            <origin xyz="0.0 0.0 0.0" rpy="0.0 0.0 0.0" />
         </xacro:inertial_cylinder>
     </link>
